File: PDB V1/Test PDB V1 11:8.kicad_sch (KiCad schematic)
At the start: 14 parts, among them J1 1805375, Q1 Q_NMOS, U1 PTPS48000QDGXRQ1, U3 XT30PW-M, U4 XT30PW-M, U5 XT30PW-M, U6 XT30PW-M

Commit message: 11/8 Final Commit of the Day
We finished the base schematic just need to upload a fuse and an NMOS part and we are good to go.
Connections:
- net GND: now also J1.1, U3.2, U4.2, U5.2, U6.2
- net at J1.2: now also F1.1
- net at U6.1: now also CBST.2, C_load.1, Q1.S, R_load.1, U1.13 (SRC), U3.1, U4.1, U5.1
- net at F1.2: now also U1.3 (INP)
Other:
- moved on the sheet: F1, J1, U3, U4, U5, U6
